Commit message: CHanges to GPS nad Map

File: robot_description/urdf/robot_core.xacro (robot description, xacro)
@@ -2,5 +2,5 @@
 <robot xmlns:xacro="http://www.ros.org/wiki/xacro">
     <!-- Macros or constants -->
-    <xacro:property name="wheel_radius" value="0.05"/>
+    <xacro:property name="wheel_radius" value="0.14"/>
     <xacro:property name="wheel_width" value="0.02"/>
     <xacro:property name="base_height" value="0.1"/>

File: robot_description/urdf/test.xacro (robot description, xacro)
@@ -1,24 +1,34 @@
 <?xml version="1.0"?>
-<robot xmlns:xacro="http://www.ros.org/wiki/xacro" name="my_custom_robot">
-  <xacro:property name="chassis_length" value="0.4" />
-  <xacro:property name="chassis_width" value="0.3" />
-  <xacro:property name="chassis_height" value="0.15" />
-  <xacro:property name="chassis_mass" value="5.0" />
-  <xacro:property name="base_color" value="White" />
-  <xacro:property name="wheel_radius" value="0.05" />
-  <xacro:property name="wheel_width" value="0.04" />
-  <xacro:property name="wheel_mass" value="0.5" />
-  <xacro:property name="wheel_color" value="Black" />
-  <xacro:property name="wheelbase_x" value="0.3" />
-  <xacro:property name="track_width" value="0.28" />
-  <xacro:property name="wheel_z_offset" value="${-chassis_height/2 + wheel_radius}" />
+<robot xmlns:xacro="http://www.ros.org/wiki/xacro" name="my_custom_robot_hardware">
+  <xacro:property name="chassis_length" value="1.0" />
+  <xacro:property name="chassis_width"  value="0.58" />
+  <xacro:property name="chassis_height" value="0.32" />
+  <xacro:property name="chassis_mass"   value="15.0" />
+  <xacro:property name="wheel_radius" value="0.14" />
+  <xacro:property name="wheel_width"  value="0.12" />
+  <xacro:property name="wheel_mass"   value="1.5" />
+  <xacro:property name="wheelbase_x"  value="0.8" />
+  <xacro:property name="track_width"  value="0.55" />
+  <xacro:property name="wheel_z_offset" value="${-chassis_height + wheel_radius}" />
   <xacro:property name="steer_link_length" value="0.02" />
   <xacro:property name="steer_link_radius" value="0.01" />
   <xacro:property name="steer_link_mass" value="0.1" />
   <xacro:property name="max_steer_angle" value="${pi/6}" />
+  <material name="PlasticWhite">
+      <color rgba="0.9 0.9 0.9 1.0"/>
+  </material>
+  <material name="PlasticBlack">
+      <color rgba="0.1 0.1 0.1 1.0"/>
+  </material>
+  <material name="PlasticRed">
+      <color rgba="0.8 0.1 0.1 1.0"/>
+  </material>
+  <material name="SensorBlue">
+      <color rgba="0.1 0.1 0.8 1.0"/>
+  </material>
   <xacro:macro name="box_inertia" params="m l w h">
-    <inertia ixx="${m/12 * (h*h + l*l)}" ixy="0.0" ixz="0.0"
-             iyy="${m/12 * (w*w + l*l)}" iyz="0.0"
-             izz="${m/12 * (w*w + h*h)}" />
+    <inertia ixx="${m/12 * (h*h + w*w)}" ixy="0.0" ixz="0.0"
+             iyy="${m/12 * (h*h + l*l)}" iyz="0.0"
+             izz="${m/12 * (w*w + l*l)}" />
   </xacro:macro>
   <xacro:macro name="cylinder_inertia" params="m r h">
@@ -32,13 +42,4 @@
              izz="${2*m/5 * r*r}" />
   </xacro:macro>
-  <material name="PlasticWhite">
-      <color rgba="0.9 0.9 0.9 1.0"/>
-  </material>
-  <material name="PlasticBlack">
-      <color rgba="0.1 0.1 0.1 1.0"/>
-  </material>
-  <material name="PlasticRed">
-      <color rgba="0.8 0.1 0.1 1.0"/>
-  </material>
   <link name="base_footprint"/>
   <link name="base_link">
@@ -57,6 +58,5 @@
     </collision>
     <inertial>
-      <origin xyz="0 0 0" rpy="0 0 0"/>
-      <mass value="${chassis_mass}"/>
+      <origin xyz="0 0 0" rpy="0 0 0"/> <mass value="${chassis_mass}"/>
       <xacro:box_inertia m="${chassis_mass}" l="${chassis_length}" w="${chassis_width}" h="${chassis_height}" />
     </inertial>
@@ -65,8 +65,7 @@
     <parent link="base_footprint"/>
     <child link="base_link"/>
-    <origin xyz="0 0 ${chassis_height/2 - wheel_z_offset}" rpy="0 0 0"/>
-  </joint>
-  <xacro:macro name="wheel" params="prefix reflect">
-    <link name="${prefix}_wheel_link">
+    <origin xyz="0 0 ${wheel_radius}" rpy="0 0 0"/>
+  </joint>
+  <xacro:macro name="wheel" params="prefix"> <link name="${prefix}_wheel_link">
       <visual>
         <origin xyz="0 0 0" rpy="${pi/2} 0 0" />
@@ -89,25 +88,20 @@
     </link>
     <joint name="${prefix}_wheel_joint" type="continuous">
-      <parent link="${prefix}_steer_link"/>
-      <child link="${prefix}_wheel_link"/>
+      <parent link="${prefix}_steer_link"/> <child link="${prefix}_wheel_link"/>
       <origin xyz="0 0 0" rpy="0 0 0"/>
-      <axis xyz="0 1 0"/>
-      <limit effort="100" velocity="100"/>
-    </joint>
+      <axis xyz="0 1 0"/> <limit effort="100" velocity="100"/> </joint>
     <transmission name="${prefix}_wheel_transmission">
       <type>transmission_interface/SimpleTransmission</type>
       <joint name="${prefix}_wheel_joint">
-        <hardwareInterface>hardware_interface/VelocityJointInterface</hardwareInterface>
+         <hardwareInterface>hardware_interface/VelocityJointInterface</hardwareInterface>
       </joint>
       <actuator name="${prefix}_wheel_motor">
-        <hardwareInterface>hardware_interface/VelocityJointInterface</hardwareInterface>
-        <mechanicalReduction>1</mechanicalReduction>
-      </actuator>
+         <hardwareInterface>hardware_interface/VelocityJointInterface</hardwareInterface>
+         <mechanicalReduction>1</mechanicalReduction> </actuator>
     </transmission>
   </xacro:macro>
   <xacro:macro name="steering_link" params="prefix reflect_steer">
     <link name="${prefix}_steer_link">
-      <visual>
-        <origin xyz="0 0 0" rpy="0 0 0" />
+      <visual> <origin xyz="0 0 0" rpy="0 0 0" />
         <geometry>
           <cylinder radius="${steer_link_radius}" length="${steer_link_length}"/>
@@ -121,6 +115,5 @@
         </geometry>
       </collision>
-      <inertial>
-        <origin xyz="0 0 0" rpy="0 0 0"/>
+      <inertial> <origin xyz="0 0 0" rpy="0 0 0"/>
         <mass value="${steer_link_mass}"/>
         <xacro:cylinder_inertia m="${steer_link_mass}" r="${steer_link_radius}" h="${steer_link_length}" />
@@ -136,96 +129,87 @@
         <type>transmission_interface/SimpleTransmission</type>
         <joint name="${prefix}_steer_joint">
-            <hardwareInterface>hardware_interface/PositionJointInterface</hardwareInterface>
+             <hardwareInterface>hardware_interface/PositionJointInterface</hardwareInterface>
         </joint>
         <actuator name="${prefix}_steer_motor">
-            <hardwareInterface>hardware_interface/PositionJointInterface</hardwareInterface>
-            <mechanicalReduction>1</mechanicalReduction>
-        </actuator>
+             <hardwareInterface>hardware_interface/PositionJointInterface</hardwareInterface>
+             <mechanicalReduction>1</mechanicalReduction> </actuator>
     </transmission>
-    <xacro:wheel prefix="${prefix}" reflect="${reflect_steer}"/>
+    <xacro:wheel prefix="${prefix}"/>
   </xacro:macro>
   <xacro:macro name="rear_wheel" params="prefix reflect">
-      <link name="${prefix}_steer_link"/> <joint name="${prefix}_dummy_fixed_joint" type="fixed">
+      <link name="${prefix}_steer_link"/>
+      <joint name="${prefix}_dummy_fixed_joint" type="fixed">
           <parent link="base_link"/>
           <child link="${prefix}_steer_link"/>
           <origin xyz="${-wheelbase_x/2} ${reflect*track_width/2} ${wheel_z_offset}" rpy="0 0 0"/>
       </joint>
-      <xacro:wheel prefix="${prefix}" reflect="${reflect}"/>
-  </xacro:macro>
-  <xacro:steering_link prefix="front_left" reflect_steer="1" />
+      <xacro:wheel prefix="${prefix}"/>
+  </xacro:macro>
+  <xacro:steering_link prefix="front_left"  reflect_steer="1" />
   <xacro:steering_link prefix="front_right" reflect_steer="-1" />
-  <xacro:rear_wheel prefix="rear_left" reflect="1" />
+  <xacro:rear_wheel prefix="rear_left"  reflect="1" />
   <xacro:rear_wheel prefix="rear_right" reflect="-1" />
-  <ros2_control name="RealRobot" type="system">
-    <hardware>
-        <plugin>gazebo_ros2_control/GazeboSystem</plugin>
-        </hardware>
-    <joint name="front_left_wheel_joint">
-        <command_interface name="velocity">
-            <param name="min">-10</param> <param name="max">10</param>  </command_interface>
-        <state_interface name="position"/>
-        <state_interface name="velocity"/>
-    </joint>
-    <joint name="front_right_wheel_joint">
-        <command_interface name="velocity">
-            <param name="min">-10</param> <param name="max">10</param>  </command_interface>
-        <state_interface name="position"/>
-        <state_interface name="velocity"/>
-    </joint>
-    <joint name="rear_left_wheel_joint">
-        <command_interface name="velocity">
-            <param name="min">-10</param> <param name="max">10</param>  </command_interface>
-        <state_interface name="position"/>
-        <state_interface name="velocity"/>
-    </joint>
-    <joint name="rear_right_wheel_joint">
-        <command_interface name="velocity">
-            <param name="min">-10</param> <param name="max">10</param>  </command_interface>
-        <state_interface name="position"/>
-        <state_interface name="velocity"/>
-    </joint>
-    <joint name="front_left_steer_joint">
-        <command_interface name="position">
-            <param name="min">${-max_steer_angle}</param> <param name="max">${max_steer_angle}</param>  </command_interface>
-        <state_interface name="position"/>
-        <state_interface name="velocity"/> </joint>
-    <joint name="front_right_steer_joint">
-        <command_interface name="position">
-            <param name="min">${-max_steer_angle}</param> <param name="max">${max_steer_angle}</param>  </command_interface>
-        <state_interface name="position"/>
-        <state_interface name="velocity"/>
-    </joint>
-  </ros2_control>
-  <gazebo>
-      <plugin filename="libgazebo_ros2_control.so" name="gazebo_ros2_control">
-          <robot_param>robot_description</robot_param>
-          <robot_param_node>robot_state_publisher</robot_param_node>
-          <parameters>$(find your_robot_description_pkg)/config/my_controllers.yaml</parameters>
-          </plugin>
-  </gazebo>
-  <gazebo reference="base_link">
-    <material>Gazebo/White</material>
-    <mu1>0.2</mu1>
-    <mu2>0.2</mu2>
-  </gazebo>
-  <gazebo reference="front_left_wheel_link">
-    <material>Gazebo/Black</material>
-    <mu1>1.0</mu1>
-    <mu2>1.0</mu2>
-  </gazebo>
-  <gazebo reference="front_right_wheel_link">
-    <material>Gazebo/Black</material>
-    <mu1>1.0</mu1>
-    <mu2>1.0</mu2>
-  </gazebo>
-  <gazebo reference="rear_left_wheel_link">
-    <material>Gazebo/Black</material>
-    <mu1>1.0</mu1>
-    <mu2>1.0</mu2>
-  </gazebo>
-  <gazebo reference="rear_right_wheel_link">
-    <material>Gazebo/Black</material>
-    <mu1>1.0</mu1>
-    <mu2>1.0</mu2>
-  </gazebo>
+  <link name="imu_link">
+     <visual>
+       <geometry>
+         <box size="0.05 0.05 0.02"/>
+       </geometry>
+        <material name="SensorBlue"/>
+     </visual>
+     <collision>
+       <geometry>
+         <box size="0.05 0.05 0.02"/>
+       </geometry>
+     </collision>
+     <inertial>
+        <mass value="0.05"/> <xacro:box_inertia m="0.05" l="0.05" w="0.05" h="0.02"/>
+     </inertial>
+  </link>
+  <joint name="imu_joint" type="fixed">
+    <parent link="base_link"/>
+    <child link="imu_link"/>
+    <origin xyz="0.05 0 ${chassis_height/2 - 0.01}" rpy="0 0 0"/>
+  </joint>
+  <link name="gps_link">
+      <visual>
+       <geometry>
+         <cylinder radius="0.04" length="0.03"/>
+       </geometry>
+       <material name="SensorBlue"/>
+     </visual>
+      <collision>
+       <geometry>
+         <cylinder radius="0.04" length="0.03"/>
+       </geometry>
+     </collision>
+     <inertial>
+        <mass value="0.08"/> <xacro:cylinder_inertia m="0.08" r="0.04" h="0.03"/>
+     </inertial>
+  </link>
+  <joint name="gps_joint" type="fixed">
+    <parent link="base_link"/>
+    <child link="gps_link"/>
+    <origin xyz="-0.2 0 ${chassis_height/2 + 0.015}" rpy="0 0 0"/>
+  </joint>
+  <link name="lidar_link">
+     <visual>
+       <geometry>
+         <cylinder radius="0.05" length="0.07"/>
+       </geometry>
+       <material name="SensorBlue"/>
+     </visual>
+     <collision>
+       <geometry>
+         <cylinder radius="0.05" length="0.07"/>
+       </geometry>
+     </collision>
+      <inertial>
+        <mass value="0.2"/> <xacro:cylinder_inertia m="0.2" r="0.05" h="0.07"/>
+     </inertial>
+  </link>
+  <joint name="lidar_joint" type="fixed">
+    <parent link="base_link"/>
+    <child link="lidar_link"/>
+    <origin xyz="${chassis_length/2 - 0.1} 0 ${chassis_height/2 + 0.035}" rpy="0 0 0"/>
+  </joint>
   </robot>
