Commit message: MAJOR UPDATES

File: cacc_description/urdf/test.xacro (robot description, xacro)
@@ -42,5 +42,5 @@
              izz="${2*m/5 * r*r}" />
   </xacro:macro>
-  <link name="base_footprint"/>
+  <link name="world_dummy_link" />
   <link name="base_link">
     <visual>
@@ -62,8 +62,8 @@
     </inertial>
   </link>
-  <joint name="base_footprint_joint" type="fixed">
-    <parent link="base_footprint"/>
+  <joint name="world_to_base_joint" type="fixed">
+    <parent link="world_dummy_link"/>
     <child link="base_link"/>
-    <origin xyz="0 0 ${wheel_radius}" rpy="0 0 0"/>
+    <origin xyz="0 0 0" rpy="0 0 0"/>
   </joint>
   <xacro:macro name="wheel" params="prefix"> <link name="${prefix}_wheel_link">
@@ -192,5 +192,5 @@
     <origin xyz="-0.2 0 ${chassis_height/2 + 0.015}" rpy="0 0 0"/>
   </joint>
-  <link name="lidar_link">
+  <link name="laser">
      <visual>
        <geometry>
@@ -210,5 +210,5 @@
   <joint name="lidar_joint" type="fixed">
     <parent link="base_link"/>
-    <child link="lidar_link"/>
+    <child link="laser"/>
     <origin xyz="${chassis_length/2 - 0.1} 0 ${chassis_height/2 + 0.035}" rpy="0 0 0"/>
   </joint>
